Commit message: 底盘模拟

File: rc2024/src/r2_arm_test_01/urdf/r2Arm.urdf (robot description, URDF)
Before this commit: robot r2Arm, 4 links, 3 joints
Joints:
- joint joint1: limit (none) -> lower=0 upper=6.28 effort=1000.0 velocity=0.5; origin xyz=0 0.18031 -0.0183 rpy=1.5703 1.5708 0 -> xyz=0 0.18031 -0.0183 rpy=-1.5708 1.5708 0; type continuous -> revolute

Commit message: r2 arm 2

File: rc2024/src/r2_arm_test_01/urdf/r2Arm.urdf (robot description, URDF)
Before this commit: robot r2Arm, 4 links, 3 joints
Joints:
- joint joint1: limit lower=0 upper=6.28 effort=1000.0 velocity=0.5 -> lower=1.0471 upper=5.23 effort=1000.0 velocity=0.5
